File: pcb/icy-gecko.sch (EAGLE design)
At the start: 4 parts, among them J1 USB-C, U1 EFM32GG12B8XX_QFN64, U2 ICE40LP384-SG32, U3 MIC23159

Commit message: sch work
Parts:
- added D1: SK9822, Opto-electronics > LED Emitters:SK9822
- added D2: B0530W, Semiconductors > Discrete Semiconductors > Diodes & Rectifiers > Schottky Diodes & Rectifiers:B0530W
- added F1: (no value), Circuit Protection > Resettable Fuses - PPTC:PTC1210
- added SW1: (no value), Eletromechanical > Switches > Tactile Switches:PUSH_BUTTON
- added U4: W25Q40BVZP, Semiconductors > Integrated Circuits - ICs > Memory ICs > Flash:W25Q40BVZP
Other:
- moved on the sheet: J1, U1, U2, U3
Changed lines of the file:
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@@
 <schematic xreflabel="%F%N/%S.%C%R" xrefpart="/%S.%C%R">
 <attributes>
+<attribute name="COMPANY" value="RST"/>
+<attribute name="CREVISION" value="1.0"/>
+<attribute name="DESIGNER" value="Rafael Silva"/>
+<attribute name="LICENSE" value="GNU General Public License v3.0"/>
+<attribute name="LINK" value="https://github.com/gimbas"/>
 </attributes>
 <variantdefs>
@@
 <part name="U2" library="Semiconductors &gt; Embedded Processors &amp; Controllers &gt; FPGA - Field Programmable Gate Array" deviceset="ICE40LP384-SG32" device=""/>
 <part name="U3" library="Power &gt; Switching Controllers" deviceset="MIC23159" device=""/>
+<part name="U4" library="Semiconductors &gt; Integrated Circuits - ICs &gt; Memory ICs &gt; Flash" deviceset="W25Q40BV" device="ZP"/>
+<part name="F1" library="Circuit Protection &gt; Resettable Fuses - PPTC" deviceset="PTC" device="1210"/>
+<part name="D1" library="Opto-electronics &gt; LED Emitters" deviceset="SK9822" device=""/>
+<part name="SW1" library="Eletromechanical &gt; Switches &gt; Tactile Switches" deviceset="PUSH_BUTTON" device=""/>
+<part name="D2" library="Semiconductors &gt; Discrete Semiconductors &gt; Diodes &amp; Rectifiers &gt; Schottky Diodes &amp; Rectifiers" deviceset="B0530W" device=""/>
+<part name="SUPPLY1" library="Utility &gt; Power Symbols" deviceset="3.3V" device=""/>
+<part name="GND1" library="Utility &gt; Power Symbols" deviceset="GND" device=""/>
+<part name="SUPPLY2" library="Utility &gt; Power Symbols" deviceset="VUSB" device=""/>
+<part name="FRAME1" library="Utility &gt; Schematic" deviceset="FRAME" device="">
+<attribute name="COMPANY" value=""/>
+<attribute name="CREVISION" value=""/>
+<attribute name="DESIGNER" value=""/>
+<attribute name="LICENSE" value=""/>
+<attribute name="LINK" value=""/>
+</part>
 </parts>
 <sheets>
@@
 </plain>
 <instances>
-<instance part="J1" gate="G$1" x="-66.04" y="63.5" smashed="yes" rot="MR0">
-<attribute name="VALUE" x="-66.04" y="60.96" size="1.778" layer="96" rot="MR0"/>
-<attribute name="NAME" x="-66.04" y="101.6" size="1.778" layer="95" rot="MR0" align="top-left"/>
+<instance part="J1" gate="G$1" x="40.64" y="119.38" smashed="yes" rot="MR0">
+<attribute name="VALUE" x="40.64" y="116.84" size="1.778" layer="96" rot="MR0"/>
+<attribute name="NAME" x="40.64" y="157.48" size="1.778" layer="95" rot="MR0" align="top-left"/>
 </instance>
-<instance part="U1" gate="G$1" x="93.98" y="170.18" smashed="yes" rot="MR0">
-<attribute name="NAME" x="127" y="172.72" size="1.27" layer="95" rot="MR0" align="top-left"/>
-<attribute name="VALUE" x="127" y="-7.62" size="1.27" layer="96" rot="MR0"/>
+<instance part="U1" gate="G$1" x="200.66" y="226.06" smashed="yes" rot="MR0">
+<attribute name="NAME" x="233.68" y="228.6" size="1.27" layer="95" rot="MR0" align="top-left"/>
+<attribute name="VALUE" x="233.68" y="48.26" size="1.27" layer="96" rot="MR0"/>
 </instance>
-<instance part="U2" gate="G$1" x="233.68" y="33.02" smashed="yes" rot="MR0">
-<attribute name="NAME" x="233.68" y="124.46" size="1.524" layer="95" rot="MR0" align="top-left"/>
-<attribute name="VALUE" x="233.68" y="30.48" size="1.524" layer="96" rot="MR0"/>
+<instance part="U2" gate="G$1" x="340.36" y="88.9" smashed="yes" rot="MR0">
+<attribute name="NAME" x="340.36" y="180.34" size="1.524" layer="95" rot="MR0" align="top-left"/>
+<attribute name="VALUE" x="340.36" y="86.36" size="1.524" layer="96" rot="MR0"/>
 </instance>
-<instance part="U3" gate="G$1" x="-10.16" y="109.22" smashed="yes" rot="MR0">
-<attribute name="NAME" x="20.32" y="112.776" size="1.27" layer="95" rot="MR0"/>
-<attribute name="VALUE" x="20.32" y="110.49" size="1.27" layer="96" rot="MR0"/>
+<instance part="U3" gate="G$1" x="96.52" y="165.1" smashed="yes" rot="MR0">
+<attribute name="NAME" x="127" y="168.656" size="1.27" layer="95" rot="MR0"/>
+<attribute name="VALUE" x="127" y="166.37" size="1.27" layer="96" rot="MR0"/>
+</instance>
+<instance part="U4" gate="G$1" x="266.7" y="68.58" smashed="yes">
+<attribute name="NAME" x="254" y="74.295" size="1.778" layer="95"/>
+<attribute name="VALUE" x="254" y="58.42" size="1.778" layer="96"/>
+</instance>
+<instance part="F1" gate="G$2" x="58.42" y="149.86" smashed="yes">
+<attribute name="NAME" x="54.61" y="153.67" size="1.27" layer="95"/>
+<attribute name="VALUE" x="54.61" y="146.05" size="1.27" layer="96"/>
+</instance>
+<instance part="D1" gate="G$1" x="58.42" y="83.82" smashed="yes">
+<attribute name="NAME" x="50.8" y="91.44" size="1.778" layer="95" align="top-left"/>
+<attribute name="VALUE" x="50.8" y="73.66" size="1.778" layer="95"/>
+</instance>
+<instance part="SW1" gate="G$1" x="109.22" y="91.44" smashed="yes">
+<attribute name="NAME" x="106.68" y="97.79" size="1.778" layer="95"/>
+<attribute name="VALUE" x="106.68" y="85.09" size="1.778" layer="96"/>
+</instance>
+<instance part="D2" gate="G$1" x="353.06" y="111.76" smashed="yes" rot="R180">
+<attribute name="NAME" x="355.346" y="109.855" size="1.778" layer="95" rot="R180"/>
+<attribute name="VALUE" x="355.346" y="115.189" size="1.778" layer="96" rot="R180"/>
+</instance>
+<instance part="SUPPLY1" gate="G$1" x="180.34" y="154.94" smashed="yes">
+<attribute name="VALUE" x="180.34" y="157.734" size="1.778" layer="96" align="bottom-center"/>
+</instance>
+<instance part="GND1" gate="1" x="172.72" y="114.3" smashed="yes">
+<attribute name="VALUE" x="172.72" y="114.046" size="1.778" layer="96" align="top-center"/>
+</instance>
+<instance part="SUPPLY2" gate="G$1" x="48.26" y="160.02" smashed="yes">
+<attribute name="VALUE" x="48.26" y="162.814" size="1.778" layer="96" align="bottom-center"/>
+</instance>
+<instance part="FRAME1" gate="G$1" x="0" y="0" smashed="yes"/>
+<instance part="FRAME1" gate="G$2" x="278.13" y="10.16" smashed="yes">
+<attribute name="LAST_DATE_TIME" x="290.322" y="11.43" size="2.54" layer="94"/>
+<attribute name="SHEET" x="363.474" y="11.43" size="2.54" layer="94"/>
+<attribute name="DRAWING_NAME" x="292.3" y="27.94" size="2.54" layer="94"/>
+<attribute name="CREVISION" x="367" y="17.68" size="2.54" layer="94"/>
+<attribute name="COMPANY" x="335.48" y="16.764" size="2.54" layer="94"/>
+<attribute name="LICENSE" x="280.67" y="5.588" size="2.159" layer="94"/>
+<attribute name="DESIGNER" x="279.6" y="16.764" size="2.54" layer="94"/>
+<attribute name="LINK" x="280.67" y="1.778" size="1.778" layer="94"/>
 </instance>
 </instances>

Commit message: finish sch, scrap pcb
Parts:
- removed U4: W25Q40BVZP, Semiconductors > Integrated Circuits - ICs > Memory ICs > Flash:W25Q40BVZP
- added C1, C19, C2, C20, C21, C22, C24, C25, C3, C4, C5, C6, C7: 100n, Passive Components > Capacitors > Multilayer Ceramic Capacitors MLCC:MLCC0603
- added C10, C13: 470p, Passive Components > Capacitors > Multilayer Ceramic Capacitors MLCC:MLCC0603
- added C11, C14, C15, C8: 10u, Passive Components > Capacitors > Multilayer Ceramic Capacitors MLCC:MLCC0603
- added C12, C17, C18, C23, C26: 4u7, Passive Components > Capacitors > Multilayer Ceramic Capacitors MLCC:MLCC0603
- added C16, C9: 1u, Passive Components > Capacitors > Multilayer Ceramic Capacitors MLCC:MLCC0603
- added D3: SP0503BAHT, Circuit Protection > ESD Suppressors \ TVS Diodes:SP0503BAHT
- added J2, J3, J4, J5: 8, Connectors > Header:8
- added J6, J7: 4, Connectors > Header:4
- added L1, L2, L3: 1u, Passive Components > Inductors, Chokes & Coils:INDUCTOR_NC_0806
- added R1, R6: 10k, Passive Components > Resistors > Chip Resistors:RESISTOR0603
- added R10, R11, R14, R17, R7: 100k, Passive Components > Resistors > Chip Resistors:RESISTOR0603
- added R12: 274k, Passive Components > Resistors > Chip Resistors:RESISTOR0603
- added R13: 294k, Passive Components > Resistors > Chip Resistors:RESISTOR0603
- added R15, R16: 5k11, Passive Components > Resistors > Chip Resistors:RESISTOR0603
- added R18, R19: 22, Passive Components > Resistors > Chip Resistors:RESISTOR0603
- added R5: 2k2, Passive Components > Resistors > Chip Resistors:RESISTOR0603
- added R8: 309k, Passive Components > Resistors > Chip Resistors:RESISTOR0603
- added R9: 71k5, Passive Components > Resistors > Chip Resistors:RESISTOR0603
- added TC1: TC2050-IDC-NL, Connectors > Other:TC2050-IDC-NL
- added U6: SST26VF016B, Microchip:SST26VF016B
- added X1: (no value), Passive Components > Frequency Control & Timing Devices > Crystals:CRYSTAL_4P
- added X2: (no value), Passive Components > Frequency Control & Timing Devices > Crystals:CRYSTAL2-SMD-3215
- F1: value (none) -> 100mA; device Circuit Protection > Resettable Fuses - PPTC:PTC1210 -> Circuit Protection > Resettable Fuses - PPTC:PTC0805
Connections:
- new net !CRESET: R6.P$2, U1.PA6@7, U2.!CRESET_B@10
- new net !MCU_RESET: R1.P$1, SW1.1, TC1-10(!RESET!).S, U1.!RESET@21
- new net 1.2V: C1.P$1, C14.P$1, J6-1.S, J7-1.S, L2.P$1, R12.P$1, U2.VCC@25, U3.SNS@0
- new net 1V2_PG: R11.P$1, U1.PC4@13, U3.PG@0
- new net 3.3V: C11.P$1, C19.P$1, C2.P$1, C20.P$1, C21.P$1, C22.P$1, C24.P$1, C26.P$1, C3.P$1, C4.P$1, C5.P$1, C6.P$1, D2.A, J6-2.S, J7-2.S, L1.P$1, R1.P$2, R11.P$2, R14.P$2, R17.P$2, R5.P$2, R8.P$2, TC1-1(VTARGET).S, U1.AVDD@24, U1.IOVDD0@27, U1.IOVDD0@55, U1.IOVDD0@8, U1.VREGVDD@38, U2.VCCIO_0@28, U2.VCCIO_1@17, U2.VCCIO_2@9, U2.VCCIO_3@4, U2.VCC_SPI@16, U3.SNS@1, U6.VCC
- new net 3V3_PG: R14.P$1, U1.PC5@14, U3.PG@1
- new net CDONE: R5.P$1, U1.PA8@17, U2.CDONE@11
- new net CLK: U1.PA12@18, U2.IOR_35_GBIN3@19
- new net DN: R19.P$2, U1.PF10@47
- new net DP: R18.P$2, U1.PF11@48
- new net GND: C1.P$2, C10.P$2, C11.P$2, C12.P$2, C13.P$2, C14.P$2, C15.P$2, C16.P$2, C17.P$2, C18.P$2, C19.P$2, C2.P$2, C20.P$2, C21.P$2, C22.P$2, C23.P$2, C24.P$2, C25.P$2, C26.P$2, C3.P$2, C4.P$2, C5.P$2, C6.P$2, C7.P$2, C8.P$2, C9.P$2, D1.GND@2, D3.1, J1.GND@A1,A12,B12,B1, J1.SHIELD, J3-1.S, J4-8.S, J6-4.S, J7-4.S, R13.P$2, R15.P$1, R16.P$1, R6.P$1, R9.P$1, SW1.3, SW1.4, TC1-3(GND).S, TC1-9(TRST).S, U1.VREGVSS@36, U1.VSS@65, U2.GND@21, U2.GND@3, U2.GND@33, U3.AGND@0, U3.AGND@1, U3.PGND@0, U3.PGND@1, U3.PGND@2, U6.GND, X1.GND@0, X1.GND@1
- new net GPRST: U1.PA13@19, U2.IOR_36_GBIN2@20
- new net IOL_2A: U2.IOL_2A@2
- new net IOL_2B: U2.IOL_2B@1
- new net IOL_4A: U2.IOL_4A@5
- new net IOL_4B_GBIN7: U2.IOL_4B_GBIN7@6
- new net IOL_5A_GBIN6: U2.IOL_5A_GBIN6@8
- new net IOL_5B: U2.IOL_5B@7
- new net IOR_34: U2.IOR_34@18
- new net IOR_38: U2.IOR_38@22
- new net IOR_39: U2.IOR_39@23
- new net IOT_45: U2.IOT_45@26
- new net IOT_47: U2.IOT_47@27
- new net IOT_49_GBIN0: U2.IOT_49_GBIN0@29
- new net IOT_50_GBIN1: U2.IOT_50_GBIN1@30
- new net IOT_52: U2.IOT_52@32
- new net IOT_53: U2.IOT_53@31
- new net LED_CLK: D1.CLKI@4, U1.PD2@30
- new net LED_MOSI: D1.SDI@3, U1.PD0@28
- new net MAIN_HFXTAL_N: U1.PB13@25, X1.1
- new net MAIN_HFXTAL_P: U1.PB14@26, X1.2
- new net MAIN_LFXTAL_N: U1.PB8@16, X2.2
- new net MAIN_LFXTAL_P: U1.PB7@15, X2.1
- new net MISO: U1.PB4@10, U2.IOB_24_SDO@12
- new net MOSI: U1.PB3@9, U2.IOB_25_SDI@13
- new net MPU_PWR: R10.P$1, U3.EN@0
- new net N$1: C7.P$1, D2.C, U2.VPP_2V5@24
- new net N$32: R7.P$1, U3.EN@1
- new net N$33: L1.P$2, U3.SW@1
- new net N$34: C10.P$1, U3.SS@1
- new net N$35: R8.P$1, R9.P$2, U3.FB@1
- new net N$36: L2.P$2, U3.SW@0
- new net N$37: C13.P$1, U3.SS@0
- new net N$38: R12.P$2, R13.P$1, U3.FB@0
- new net N$39: C17.P$1, U1.VREGO@46
- new net N$40: F1.2, J1.VBUS@A4,A9,B9,B4
- new net N$41: J1.CC2@B5, R15.P$2
- new net N$42: J1.CC1@A5, R16.P$2
- new net N$43: L3.P$1, U1.VREGSW@37
- new net N$45: C23.P$1, U1.DECOUPLE@40
- new net N$48: C18.P$1, L3.P$2, U1.DVDD@39
- new net PD3: U1.PD3@31
- new net PD4: U1.PD4@32
- new net PD5: U1.PD5@33
- new net PD6: U1.PD6@34
- new net PE10: U1.PE10@58
- new net PE11: U1.PE11@59
- new net PE12: U1.PE12@60
- new net PE13: U1.PE13@61
- new net PE4: U1.PE4@41
- new net PE5: U1.PE5@42
- new net PE6: U1.PE6@43
- new net PE7: U1.PE7@44
- new net PE8: U1.PE8@56
- new net PE9: U1.PE9@57
- new net PF12: U1.PF12@53
- new net QSPI_CLK: U1.PE14@62, U6.SCK
- new net QSPI_CS0: R17.P$1, U1.PA0@1, U6.!CS!
- new net QSPI_D0: U1.PA2@3, U6.MOSI/IO0
- new net QSPI_D1: U1.PA3@4, U6.MISO/IO1
- new net QSPI_D2: U1.PA4@5, U6.!WP!/IO2
- new net QSPI_D3: U1.PA5@6, U6.!HOLD!/IO3
- new net SCK: U1.PB5@11, U2.IOB_26_SCK@15
- new net SS: U1.PB6@12, U2.IOB_27_SS@14
- new net SWCLK: TC1-4(TCK/SWCLK).S, U1.PF0@49
- new net SWDIO: TC1-2(TMS/SWDIO).S, U1.PF1@50
- new net SWO: TC1-6(TDO/SWO).S, U1.PF2@51
- new net USBDN: D3.4, J1.DN@A7,B7, R19.P$1
- new net USBDP: D3.3, J1.DP@A6,B6, R18.P$1
- new net VUSB: C12.P$1, C15.P$1, C16.P$1, C25.P$1, C8.P$1, C9.P$1, D1.VDD@5, D3.2, F1.1, J6-3.S, J7-3.S, R10.P$2, R7.P$2, U1.VBUS@52, U3.AVIN@0, U3.AVIN@1, U3.VIN@0, U3.VIN@1
Other:
- note added: "Pin 1"
- note added: "Pin 20"
- note added: "Pin 6"
- note added: "Pin 7"
- note added: "R1"
- note added: "R2"
- note added: "Vout = Vref*(1+(R1/R2)) Vo | R1 | R2 1V2 | 274k | 294k 1V5 | 316k | 221k 1V8 | 301k | 158k 2V5 | 324k | 107k 3V3 | 309k | 71k5"

Commit message: pcd finito
Connections:
- net 1V2_PG: now also U1.PD1@29; no longer U1.PC4@13
- net 3V3_PG: now also U1.PD8@35; no longer U1.PC5@14
- net IOL_2A: now also J4-5.S
- net IOL_2B: now also J4-6.S
- net IOL_4A: now also J4-4.S
- net IOL_4B_GBIN7: now also J4-3.S
- net IOL_5A_GBIN6: now also J4-1.S
- net IOL_5B: now also J4-2.S
- net IOR_34: now also J2-1.S
- net IOR_38: now also J2-2.S
- net IOR_39: now also J2-3.S
- net IOT_45: now also J2-4.S
- net IOT_47: now also J2-5.S
- net IOT_49_GBIN0: now also J2-6.S
- net IOT_50_GBIN1: now also J2-7.S
- net IOT_52: now also J4-7.S
- net IOT_53: now also J2-8.S
- net PD3: now also J3-2.S
- net PD4: now also J3-3.S
- net PD5: now also J3-4.S
- net PD6: now also J3-5.S
- net PE10: now also J5-4.S
- net PE11: now also J5-3.S
- net PE12: now also J5-2.S
- net PE13: now also J5-1.S
- net PE4: now also J3-6.S
- net PE5: now also J3-7.S
- net PE6: now also J5-8.S
- net PE7: now also J5-7.S
- net PE8: now also J5-6.S
- net PE9: now also J5-5.S
- net PF12: now also J3-8.S
- net USBDP: now also D3.2; no longer D3.3
- net VUSB: now also D3.3; no longer D3.2

Commit message: sync
Connections:
- net IOL_4A renamed IOL4A
- net IOL_4B_GBIN7 renamed IOL4BG7
- net IOL_5A_GBIN6 renamed IOL5AG6
- net IOL_5B renamed IOL5B
- net IOR_34 renamed IOR34
- net IOR_38 renamed IOR38
- net IOR_39 renamed IOR39
- net IOT_45 renamed IOT45
- net IOT_47 renamed IOT47
- net IOT_49_GBIN0 renamed IOT49G0
- net IOT_50_GBIN1 renamed IOT50G1
- net IOT_52 renamed IOT52
- net IOT_53 renamed IOT53
Changed lines of the file:
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@@
 </segment>
 </net>
-<net name="IOT_45" class="0">
+<net name="IOT45" class="0">
 <segment>
 <wire x1="231.14" y1="154.94" x2="233.68" y2="154.94" width="0.1524" layer="91"/>
@@
 </segment>
 </net>
-<net name="IOT_47" class="0">
+<net name="IOT47" class="0">
 <segment>
 <wire x1="233.68" y1="149.86" x2="231.14" y2="149.86" width="0.1524" layer="91"/>
@@
 </segment>
 </net>
-<net name="IOT_49_GBIN0" class="0">
+<net name="IOT49G0" class="0">
 <segment>
 <wire x1="233.68" y1="144.78" x2="231.14" y2="144.78" width="0.1524" layer="91"/>
@@
 </segment>
 </net>
-<net name="IOT_50_GBIN1" class="0">
+<net name="IOT50G1" class="0">
 <segment>
 <wire x1="233.68" y1="142.24" x2="231.14" y2="142.24" width="0.1524" layer="91"/>
@@
 </segment>
 </net>
-<net name="IOT_52" class="0">
+<net name="IOT52" class="0">
 <segment>
 <wire x1="233.68" y1="137.16" x2="231.14" y2="137.16" width="0.1524" layer="91"/>
@@
 </segment>
 </net>
-<net name="IOT_53" class="0">
+<net name="IOT53" class="0">
 <segment>
 <wire x1="233.68" y1="134.62" x2="231.14" y2="134.62" width="0.1524" layer="91"/>
@@
 </segment>
 </net>
-<net name="IOR_38" class="0">
+<net name="IOR38" class="0">
 <segment>
 <wire x1="233.68" y1="114.3" x2="231.14" y2="114.3" width="0.1524" layer="91"/>
@@
 </segment>
 </net>
-<net name="IOR_39" class="0">
+<net name="IOR39" class="0">
 <segment>
 <wire x1="231.14" y1="111.76" x2="233.68" y2="111.76" width="0.1524" layer="91"/>
@@
 </segment>
 </net>
-<net name="IOL_4A" class="0">
+<net name="IOL4A" class="0">
 <segment>
 <wire x1="233.68" y1="93.98" x2="231.14" y2="93.98" width="0.1524" layer="91"/>
@@
 </segment>
 </net>
-<net name="IOL_4B_GBIN7" class="0">
+<net name="IOL4BG7" class="0">
 <segment>
 <wire x1="233.68" y1="91.44" x2="231.14" y2="91.44" width="0.1524" layer="91"/>
@@
 </segment>
 </net>
-<net name="IOL_5A_GBIN6" class="0">
+<net name="IOL5AG6" class="0">
 <segment>
 <wire x1="233.68" y1="88.9" x2="231.14" y2="88.9" width="0.1524" layer="91"/>
@@
 </segment>
 </net>
-<net name="IOL_5B" class="0">
+<net name="IOL5B" class="0">
 <segment>
 <wire x1="233.68" y1="86.36" x2="231.14" y2="86.36" width="0.1524" layer="91"/>
@@
 </segment>
 </net>
-<net name="IOR_34" class="0">
+<net name="IOR34" class="0">
 <segment>
 <pinref part="U2" gate="G$1" pin="IOR_34@18"/>
@@
 </segment>
 </net>
-<net name="IOL_4A" class="0">
+<net name="IOL4A" class="0">
 <segment>
 <wire x1="236.22" y1="101.6" x2="236.22" y2="99.06" width="0.1524" layer="91"/>
@@
 </segment>
 </net>
-<net name="IOL_4B_GBIN7" class="0">
+<net name="IOL4BG7" class="0">
 <segment>
 <wire x1="238.76" y1="101.6" x2="238.76" y2="99.06" width="0.1524" layer="91"/>
@@
 </segment>
 </net>
-<net name="IOL_5A_GBIN6" class="0">
+<net name="IOL5AG6" class="0">
 <segment>
 <wire x1="243.84" y1="101.6" x2="243.84" y2="99.06" width="0.1524" layer="91"/>
@@
 </segment>
 </net>
-<net name="IOL_5B" class="0">
+<net name="IOL5B" class="0">
 <segment>
 <wire x1="241.3" y1="101.6" x2="241.3" y2="99.06" width="0.1524" layer="91"/>
@@
 </segment>
 </net>
-<net name="IOT_52" class="0">
+<net name="IOT52" class="0">
 <segment>
 <wire x1="228.6" y1="101.6" x2="228.6" y2="99.06" width="0.1524" layer="91"/>
@@
 </segment>
 </net>
-<net name="IOT_45" class="0">
+<net name="IOT45" class="0">
 <segment>
 <wire x1="236.22" y1="160.02" x2="236.22" y2="157.48" width="0.1524" layer="91"/>
@@
 </segment>
 </net>
-<net name="IOT_47" class="0">
+<net name="IOT47" class="0">
 <segment>
 <wire x1="233.68" y1="157.48" x2="233.68" y2="160.02" width="0.1524" layer="91"/>
@@
 </segment>
 </net>
-<net name="IOT_49_GBIN0" class="0">
+<net name="IOT49G0" class="0">
 <segment>
 <wire x1="231.14" y1="157.48" x2="231.14" y2="160.02" width="0.1524" layer="91"/>
@@
 </segment>
 </net>
-<net name="IOT_50_GBIN1" class="0">
+<net name="IOT50G1" class="0">
 <segment>
 <wire x1="228.6" y1="157.48" x2="228.6" y2="160.02" width="0.1524" layer="91"/>
@@
 </segment>
 </net>
-<net name="IOT_53" class="0">
+<net name="IOT53" class="0">
 <segment>
 <wire x1="226.06" y1="157.48" x2="226.06" y2="160.02" width="0.1524" layer="91"/>
@@
 </segment>
 </net>
-<net name="IOR_38" class="0">
+<net name="IOR38" class="0">
 <segment>
 <wire x1="241.3" y1="157.48" x2="241.3" y2="160.02" width="0.1524" layer="91"/>
@@
 </segment>
 </net>
-<net name="IOR_34" class="0">
+<net name="IOR34" class="0">
 <segment>
 <wire x1="243.84" y1="160.02" x2="243.84" y2="157.48" width="0.1524" layer="91"/>
@@
 </segment>
 </net>
-<net name="IOR_39" class="0">
+<net name="IOR39" class="0">
 <segment>
 <wire x1="238.76" y1="160.02" x2="238.76" y2="157.48" width="0.1524" layer="91"/>
