File: pcb/icy-gecko.sch (EAGLE design)
At the start: 64 parts, among them J1 USB-C, J2 8, J3 8, J4 8, J5 8, J6 4, J7 4, U1 EFM32GG12B8XX_QFN64, U2 ICE40LP384-SG32, U3 MIC23159, U6 SST26VF016B

Commit message: corrected some pcb errors
Parts:
- removed J1: USB-C, Connectors > USB:USB-C
- added USB1: USB-C-16P-SMD-FLAT-SIDE-TYPE-2, Connectors > USB:USB-C-16P-SMD-FLAT-SIDE-TYPE-2
- L3: value 1u -> 4u7
Connections:
- net GND: now also USB1.GND, USB1.SHIELD@0, USB1.SHIELD@1, USB1.SHIELD@2, USB1.SHIELD@3; no longer J1.GND@A1,A12,B12,B1, J1.SHIELD
- net N$40: now also USB1.VBUS; no longer J1.VBUS@A4,A9,B9,B4
- net N$41: now also USB1.SB2; no longer J1.CC2@B5
- net N$42: now also USB1.SB1; no longer J1.CC1@A5
- net USBDN: now also USB1.D-; no longer J1.DN@A7,B7
- net USBDP: now also USB1.D+; no longer J1.DP@A6,B6
Other:
- moved on the sheet: R18
Changed lines of the file:
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@@
 <?xml version="1.0" encoding="utf-8"?>
 <!DOCTYPE eagle SYSTEM "eagle.dtd">
-<eagle version="9.3.0">
+<eagle version="9.5.1">
 <drawing>
 <settings>
@@
 <part name="GND1" library="Utility &gt; Power Symbols" deviceset="GND" device=""/>
 <part name="GND23" library="Utility &gt; Power Symbols" deviceset="GND" device=""/>
-<part name="L3" library="Passive Components &gt; Inductors, Chokes &amp; Coils" deviceset="INDUCTOR_NC" device="_0806" value="1u"/>
+<part name="L3" library="Passive Components &gt; Inductors, Chokes &amp; Coils" deviceset="INDUCTOR_NC" device="_0806" value="4u7"/>
 <part name="C18" library="Passive Components &gt; Capacitors &gt; Multilayer Ceramic Capacitors MLCC" deviceset="MLCC" device="0603" value="4u7"/>
 <part name="GND24" library="Utility &gt; Power Symbols" deviceset="GND" device=""/>
@@
 <part name="SUPPLY17" library="Utility &gt; Power Symbols" deviceset="3.3V" device=""/>
 <part name="GND31" library="Utility &gt; Power Symbols" deviceset="GND" device=""/>
-<part name="J1" library="Connectors &gt; USB" deviceset="USB-C" device=""/>
 <part name="SUPPLY2" library="Utility &gt; Power Symbols" deviceset="VUSB" device=""/>
 <part name="F1" library="Circuit Protection &gt; Resettable Fuses - PPTC" deviceset="PTC" device="0805" value="100mA"/>
@@
 <part name="R1" library="Passive Components &gt; Resistors &gt; Chip Resistors" deviceset="RESISTOR" device="0603" value="10k"/>
 <part name="SUPPLY29" library="Utility &gt; Power Symbols" deviceset="3.3V" device=""/>
+<part name="USB1" library="Connectors &gt; USB" deviceset="USB-C-16P-SMD-FLAT-SIDE" device="-TYPE-2"/>
+<part name="GND40" library="Utility &gt; Power Symbols" deviceset="GND" device=""/>
 </parts>
 <sheets>
@@
 </plain>
 <instances>
-<instance part="J1" gate="G$1" x="91.44" y="114.3" smashed="yes" rot="MR0">
-<attribute name="VALUE" x="91.44" y="111.76" size="1.778" layer="96" rot="MR0"/>
-<attribute name="NAME" x="91.44" y="152.4" size="1.778" layer="95" rot="MR0" align="top-left"/>
-</instance>
 <instance part="SUPPLY2" gate="G$1" x="116.84" y="149.86" smashed="yes">
 <attribute name="VALUE" x="116.84" y="152.654" size="1.778" layer="96" align="bottom-center"/>
@@
 <attribute name="VALUE" x="297.18" y="119.126" size="1.778" layer="96" align="top-center"/>
 </instance>
-<instance part="R18" gate="G$1" x="124.46" y="142.24" smashed="yes">
-<attribute name="NAME" x="121.158" y="143.764" size="1.27" layer="95"/>
-<attribute name="VALUE" x="120.904" y="139.7" size="1.27" layer="96"/>
+<instance part="R18" gate="G$1" x="127" y="137.16" smashed="yes">
+<attribute name="NAME" x="123.698" y="138.684" size="1.27" layer="95"/>
+<attribute name="VALUE" x="123.444" y="134.62" size="1.27" layer="96"/>
 </instance>
 <instance part="R19" gate="G$1" x="134.62" y="139.7" smashed="yes">
@@
 <instance part="SUPPLY20" gate="G$1" x="271.78" y="134.62" smashed="yes">
 <attribute name="VALUE" x="271.78" y="137.414" size="1.778" layer="96" align="bottom-center"/>
+</instance>
+<instance part="USB1" gate="G$1" x="86.36" y="144.78" smashed="yes">
+<attribute name="NAME" x="72.136" y="121.92" size="1.27" layer="95" rot="R90"/>
+</instance>
+<instance part="GND40" gate="1" x="68.58" y="142.24" smashed="yes">
+<attribute name="VALUE" x="68.58" y="141.986" size="1.778" layer="96" align="top-center"/>
 </instance>
 </instances>
@@
 <net name="GND" class="0">
 <segment>
-<pinref part="J1" gate="G$1" pin="SHIELD"/>
-<wire x1="93.98" y1="116.84" x2="96.52" y2="116.84" width="0.1524" layer="91"/>
 <wire x1="96.52" y1="116.84" x2="96.52" y2="109.22" width="0.1524" layer="91"/>
-<pinref part="J1" gate="G$1" pin="GND@A1,A12,B12,B1"/>
-<wire x1="93.98" y1="119.38" x2="96.52" y2="119.38" width="0.1524" layer="91"/>
-<wire x1="96.52" y1="119.38" x2="96.52" y2="116.84" width="0.1524" layer="91"/>
+<wire x1="96.52" y1="124.46" x2="96.52" y2="116.84" width="0.1524" layer="91"/>
 <junction x="96.52" y="116.84"/>
 <pinref part="GND19" gate="1" pin="GND"/>
+<pinref part="USB1" gate="G$1" pin="GND"/>
+<wire x1="88.9" y1="124.46" x2="96.52" y2="124.46" width="0.1524" layer="91"/>
+<pinref part="USB1" gate="G$1" pin="SHIELD@2"/>
+<wire x1="81.28" y1="119.38" x2="81.28" y2="116.84" width="0.1524" layer="91"/>
+<wire x1="81.28" y1="116.84" x2="83.82" y2="116.84" width="0.1524" layer="91"/>
+<pinref part="USB1" gate="G$1" pin="SHIELD@1"/>
+<wire x1="83.82" y1="116.84" x2="96.52" y2="116.84" width="0.1524" layer="91"/>
+<wire x1="83.82" y1="119.38" x2="83.82" y2="116.84" width="0.1524" layer="91"/>
+<junction x="83.82" y="116.84"/>
 </segment>
 <segment>
@@
 <pinref part="J7" gate="-4" pin="S"/>
 <wire x1="162.56" y1="101.6" x2="162.56" y2="104.14" width="0.1524" layer="91"/>
+</segment>
+<segment>
+<pinref part="USB1" gate="G$1" pin="SHIELD@3"/>
+<pinref part="USB1" gate="G$1" pin="SHIELD@0"/>
+<wire x1="83.82" y1="147.32" x2="83.82" y2="149.86" width="0.1524" layer="91"/>
+<wire x1="83.82" y1="149.86" x2="81.28" y2="149.86" width="0.1524" layer="91"/>
+<junction x="81.28" y="149.86"/>
+<wire x1="81.28" y1="149.86" x2="81.28" y2="147.32" width="0.1524" layer="91"/>
+<wire x1="81.28" y1="149.86" x2="68.58" y2="149.86" width="0.1524" layer="91"/>
+<wire x1="68.58" y1="149.86" x2="68.58" y2="144.78" width="0.1524" layer="91"/>
+<pinref part="GND40" gate="1" pin="GND"/>
 </segment>
 </net>
@@
 <net name="N$40" class="0">
 <segment>
-<pinref part="J1" gate="G$1" pin="VBUS@A4,A9,B9,B4"/>
-<wire x1="93.98" y1="147.32" x2="96.52" y2="147.32" width="0.1524" layer="91"/>
 <pinref part="F1" gate="G$1" pin="2"/>
+<pinref part="USB1" gate="G$1" pin="VBUS"/>
+<wire x1="88.9" y1="142.24" x2="88.9" y2="147.32" width="0.1524" layer="91"/>
+<wire x1="88.9" y1="147.32" x2="96.52" y2="147.32" width="0.1524" layer="91"/>
 </segment>
 </net>
 <net name="N$41" class="0">
 <segment>
-<pinref part="J1" gate="G$1" pin="CC2@B5"/>
-<wire x1="93.98" y1="124.46" x2="101.6" y2="124.46" width="0.1524" layer="91"/>
-<wire x1="101.6" y1="124.46" x2="101.6" y2="121.92" width="0.1524" layer="91"/>
+<wire x1="88.9" y1="127" x2="101.6" y2="127" width="0.1524" layer="91"/>
+<wire x1="101.6" y1="127" x2="101.6" y2="121.92" width="0.1524" layer="91"/>
 <pinref part="R15" gate="G$1" pin="P$2"/>
+<pinref part="USB1" gate="G$1" pin="SB2"/>
 </segment>
 </net>
 <net name="N$42" class="0">
 <segment>
-<pinref part="J1" gate="G$1" pin="CC1@A5"/>
-<wire x1="93.98" y1="127" x2="109.22" y2="127" width="0.1524" layer="91"/>
-<wire x1="109.22" y1="127" x2="109.22" y2="121.92" width="0.1524" layer="91"/>
+<wire x1="88.9" y1="129.54" x2="109.22" y2="129.54" width="0.1524" layer="91"/>
+<wire x1="109.22" y1="129.54" x2="109.22" y2="121.92" width="0.1524" layer="91"/>
 <pinref part="R16" gate="G$1" pin="P$2"/>
+<pinref part="USB1" gate="G$1" pin="SB1"/>
 </segment>
 </net>
@@
 <net name="DP" class="0">
 <segment>
-<label x="142.24" y="142.24" size="0.889" layer="95" xref="yes"/>
-<wire x1="129.54" y1="142.24" x2="142.24" y2="142.24" width="0.1524" layer="91"/>
+<label x="142.24" y="137.16" size="0.889" layer="95" xref="yes"/>
+<wire x1="132.08" y1="137.16" x2="142.24" y2="137.16" width="0.1524" layer="91"/>
 <pinref part="R18" gate="G$1" pin="P$2"/>
 </segment>
@@
 <net name="USBDN" class="0">
 <segment>
-<pinref part="J1" gate="G$1" pin="DN@A7,B7"/>
-<wire x1="93.98" y1="139.7" x2="119.38" y2="139.7" width="0.1524" layer="91"/>
+<wire x1="88.9" y1="139.7" x2="119.38" y2="139.7" width="0.1524" layer="91"/>
 <pinref part="D3" gate="G$1" pin="4"/>
 <wire x1="119.38" y1="124.46" x2="119.38" y2="139.7" width="0.1524" layer="91"/>
@@
 <junction x="119.38" y="139.7"/>
 <pinref part="R19" gate="G$1" pin="P$1"/>
+<pinref part="USB1" gate="G$1" pin="D-"/>
 </segment>
 </net>
 <net name="USBDP" class="0">
 <segment>
-<pinref part="J1" gate="G$1" pin="DP@A6,B6"/>
-<wire x1="93.98" y1="142.24" x2="114.3" y2="142.24" width="0.1524" layer="91"/>
+<wire x1="88.9" y1="137.16" x2="114.3" y2="137.16" width="0.1524" layer="91"/>
 <pinref part="R18" gate="G$1" pin="P$1"/>
 <pinref part="D3" gate="G$1" pin="2"/>
-<wire x1="114.3" y1="142.24" x2="119.38" y2="142.24" width="0.1524" layer="91"/>
-<wire x1="114.3" y1="124.46" x2="114.3" y2="142.24" width="0.1524" layer="91"/>
-<junction x="114.3" y="142.24"/>
-</segment>
-</net>
+<wire x1="114.3" y1="137.16" x2="121.92" y2="137.16" width="0.1524" layer="91"/>
+<wire x1="114.3" y1="124.46" x2="114.3" y2="137.16" width="0.1524" layer="91"/>
+<junction x="114.3" y="137.16"/>
+<pinref part="USB1" gate="G$1" pin="D+"/>
+</segment>
+</net>
